File: hardware/pcb-v1/routed/rfid_carrier_v01.kicad_pcb (KiCad board)
At the start: 2 copper layers, 128 x 58 mm, 40 parts, among them J1 5V DC INPUT, J2 RC522, J3 LCD1602 PARALLEL, J4 STATUS LEDs, J5 5V ACTIVE BUZZER, J6 DevKit V1 socket 1x15, J7 DevKit V1 socket 1x15, Q1 BC337-40, U1 SN74AHCT244N

Commit message: feat(hardware): finish PCB V0.2 with GND pour, silk marks and Gerbers
Add GND pours on both layers, assembly marks on F.SilkS (pin-1 dots,
electrolytic +, D1 cathode bar, Q1 C/B/E), trim the dangling GPIO22
tail and export Gerber/Excellon files, DRC report, render and 1:1 SVG.

Co-Authored-By: Claude Opus 5.5 <noreply@anthropic.com>
Routing:
- net GPIO22: track 246.1 -> 233.4 mm
- added copper zone on B.Cu, net GND
- added copper zone on F.Cu, net GND
Other:
- board text added: "+"
- board text added: "5V DC ONLY"
- board text added: "ANTENNA"
- board text added: "ASSEMBLY MARK"
- board text added: "B"
- board text added: "C"
- board text added: "E"
- board text added: "ESP32 DEVKIT V1 / 30 PIN"
- board text added: "NO COPPER"
- board text added: "RFID CARRIER V0.2"
- board text added: "USB <"
Changed lines of the file:
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@@
 (via (at 84.80000000000001 71.9) (size 1) (drill .5) (layers "F.Cu" "B.Cu") (net 14))
 (segment (start 84.800000 71.900000) (end 84.800000 71.800000) (width 0.25) (layer "F.Cu") (net 14))
-(segment (start 84.800000 71.800000) (end 83.900000 70.900000) (width 0.25) (layer "F.Cu") (net 14))
+(segment (start 84.800000 71.800000) (end 83.850000 70.850000) (width 0.25) (layer "F.Cu") (net 14))
 (segment (start 24.800000 75.800000) (end 22.300000 78.300000) (width 0.5) (layer "B.Cu") (net 6))
 (via (at 22.3 78.30000000000001) (size 1) (drill .5) (layers "F.Cu" "B.Cu") (net 6))
@@
 (segment (start 103.000000 57.000000) (end 101.100000 57.000000) (width 0.2) (layer "B.Cu") (net 19))
 (segment (start 101.100000 57.000000) (end 100.800000 57.300000) (width 0.2) (layer "B.Cu") (net 19))
-(segment (start 87.000000 67.700000) (end 78.748300 75.951700) (width 0.300000) (layer "F.Cu") (net 14))
-(segment (start 78.748300 75.951700) (end 78.748300 81.255700) (width 0.300000) (layer "F.Cu") (net 14))
-(segment (start 78.748300 81.255700) (end 78.948900 81.456300) (width 0.300000) (layer "F.Cu") (net 14))
+(segment (start 87.000000 67.700000) (end 83.850000 70.850000) (width 0.300000) (layer "F.Cu") (net 14))
+(zone (net 7) (net_name "GND") (layer "F.Cu")
+   (name "GND pour F.Cu") (hatch edge 0.5) (connect_pads (clearance 0.2)) (min_thickness 0.2)
+   (filled_areas_thickness no) (fill yes (thermal_gap 0.25) (thermal_bridge_width 0.4) (island_removal_mode 0))
+   (polygon (pts (xy 4.5 39.5) (xy 131.5 39.5) (xy 131.5 96.5) (xy 4.5 96.5)))
 )
+(zone (net 7) (net_name "GND") (layer "B.Cu")
+   (name "GND pour B.Cu") (hatch edge 0.5) (connect_pads (clearance 0.2)) (min_thickness 0.2)
+   (filled_areas_thickness no) (fill yes (thermal_gap 0.25) (thermal_bridge_width 0.4) (island_removal_mode 0))
+   (polygon (pts (xy 4.5 39.5) (xy 131.5 39.5) (xy 131.5 96.5) (xy 4.5 96.5)))
+)
+(gr_text "RFID CARRIER V0.2" (at 28 52) (layer "F.SilkS") (effects (font (size 1 1) (thickness .15))))
+(gr_text "ESP32 DEVKIT V1 / 30 PIN" (at 28 55) (layer "F.SilkS") (effects (font (size 0.8 0.8) (thickness .15))))
+(gr_text "USB <" (at 20 59) (layer "F.SilkS") (effects (font (size 1 1) (thickness .15))))
+(gr_text "ANTENNA" (at 62.5 54) (layer "F.SilkS") (effects (font (size 1 1) (thickness .15))))
+(gr_text "NO COPPER" (at 62.5 57) (layer "F.SilkS") (effects (font (size 1 1) (thickness .15))))
+(gr_text "5V DC ONLY" (at 129.5 61.5 90) (layer "F.SilkS") (effects (font (size 1 1) (thickness .15))))
+(gr_text "ASSEMBLY MARK" (at 68 103) (layer "Dwgs.User") (effects (font (size 0.8 0.8) (thickness 0.12))))
+(gr_circle (center 123.05 59.00) (end 123.35 59.00) (stroke (width 0.15) (type solid)) (fill solid) (layer "F.SilkS"))
+(gr_circle (center 84.45 43.00) (end 84.75 43.00) (stroke (width 0.15) (type solid)) (fill solid) (layer "F.SilkS"))
+(gr_circle (center 85.45 87.00) (end 85.75 87.00) (stroke (width 0.15) (type solid)) (fill solid) (layer "F.SilkS"))
+(gr_circle (center 108.45 43.00) (end 108.75 43.00) (stroke (width 0.15) (type solid)) (fill solid) (layer "F.SilkS"))
+(gr_circle (center 122.45 43.00) (end 122.75 43.00) (stroke (width 0.15) (type solid)) (fill solid) (layer "F.SilkS"))
+(gr_circle (center 10.77 42.30) (end 11.07 42.30) (stroke (width 0.15) (type solid)) (fill solid) (layer "F.SilkS"))
+(gr_circle (center 10.77 67.70) (end 11.07 67.70) (stroke (width 0.15) (type solid)) (fill solid) (layer "F.SilkS"))
+(gr_circle (center 78.45 77.00) (end 78.75 77.00) (stroke (width 0.15) (type solid)) (fill solid) (layer "F.SilkS"))
+(gr_circle (center 85.45 55.00) (end 85.75 55.00) (stroke (width 0.15) (type solid)) (fill solid) (layer "F.SilkS"))
+(gr_circle (center 98.45 55.00) (end 98.75 55.00) (stroke (width 0.15) (type solid)) (fill solid) (layer "F.SilkS"))
+(gr_circle (center 101.31 79.00) (end 101.61 79.00) (stroke (width 0.15) (type solid)) (fill solid) (layer "F.SilkS"))
+(gr_text "+" (at 121.30 81.00) (layer "F.SilkS") (effects (font (size 1.2 1.2) (thickness 0.2))))
+(gr_text "+" (at 92.30 47.40) (layer "F.SilkS") (effects (font (size 1.2 1.2) (thickness 0.2))))
+(gr_text "+" (at 29.30 75.00) (layer "F.SilkS") (effects (font (size 1.2 1.2) (thickness 0.2))))
+(gr_line (start 111.55 47.00) (end 111.55 49.00) (stroke (width 0.3) (type solid)) (layer "F.SilkS"))
+(gr_text "C" (at 114.40 54.50) (layer "F.SilkS") (effects (font (size 0.8 0.8) (thickness 0.15))))
+(gr_text "B" (at 116.94 54.50) (layer "F.SilkS") (effects (font (size 0.8 0.8) (thickness 0.15))))
+(gr_text "E" (at 119.48 54.50) (layer "F.SilkS") (effects (font (size 0.8 0.8) (thickness 0.15))))
+)
